File: matrix.kicad_sch (KiCad schematic)
At the start: 66 parts

Commit message: Added LCSC, but going to switch to 0603 or 0804 components as I want to keep handsoldering an option
Parts:
- D1, D10, D11, D12, D13, D14, D15, D16, D17, D18, D19, D2, D20, D21, D3, D4, D5, D6, D7, D8, D9: LCSC (none) -> C28646371
- LED1, LED10, LED11, LED12, LED13, LED14, LED15, LED16, LED17, LED18, LED19, LED2, LED20, LED21, LED3, LED4, LED5, LED6, LED7, LED8, LED9: LCSC (none) -> C5242955
- MX1, MX10, MX11, MX12, MX13, MX14, MX15, MX16, MX17, MX18, MX19, MX2, MX20, MX21, MX3, MX4, MX5, MX6, MX7, MX8, MX9: LCSC (none) -> C5156480

Commit message: Switched to 0805 for R C and SOD-123 for Diodes
Parts:
- D1, D10, D11, D12, D13, D14, D15, D16, D17, D18, D19, D2, D20, D21, D3, D4, D5, D6, D7, D8, D9: footprint Diode_SMD:D_0402_1005Metric_Pad0.77x0.64mm_HandSolder -> ScottoKeebs_Components:Diode_SOD-123
Changed lines of the file:
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@@
 			)
 		)
-		(property "Footprint" "Diode_SMD:D_0402_1005Metric_Pad0.77x0.64mm_HandSolder"
+		(property "Footprint" "ScottoKeebs_Components:Diode_SOD-123"
 			(at 55.88 55.88 0)
 			(effects
@@
 			)
 		)
-		(property "Footprint" "Diode_SMD:D_0402_1005Metric_Pad0.77x0.64mm_HandSolder"
+		(property "Footprint" "ScottoKeebs_Components:Diode_SOD-123"
 			(at 73.66 40.64 0)
 			(effects
@@
 			)
 		)
-		(property "Footprint" "Diode_SMD:D_0402_1005Metric_Pad0.77x0.64mm_HandSolder"
+		(property "Footprint" "ScottoKeebs_Components:Diode_SOD-123"
 			(at 91.44 72.39 0)
 			(effects
@@
 			)
 		)
-		(property "Footprint" "Diode_SMD:D_0402_1005Metric_Pad0.77x0.64mm_HandSolder"
+		(property "Footprint" "ScottoKeebs_Components:Diode_SOD-123"
 			(at 109.22 80.01 0)
 			(effects
@@
 			)
 		)
-		(property "Footprint" "Diode_SMD:D_0402_1005Metric_Pad0.77x0.64mm_HandSolder"
+		(property "Footprint" "ScottoKeebs_Components:Diode_SOD-123"
 			(at 67.31 120.65 0)
 			(effects
@@
 			)
 		)
-		(property "Footprint" "Diode_SMD:D_0402_1005Metric_Pad0.77x0.64mm_HandSolder"
+		(property "Footprint" "ScottoKeebs_Components:Diode_SOD-123"
 			(at 73.66 72.39 0)
 			(effects
@@
 			)
 		)
-		(property "Footprint" "Diode_SMD:D_0402_1005Metric_Pad0.77x0.64mm_HandSolder"
+		(property "Footprint" "ScottoKeebs_Components:Diode_SOD-123"
 			(at 109.22 55.88 0)
 			(effects
@@
 			)
 		)
-		(property "Footprint" "Diode_SMD:D_0402_1005Metric_Pad0.77x0.64mm_HandSolder"
+		(property "Footprint" "ScottoKeebs_Components:Diode_SOD-123"
 			(at 109.22 113.03 0)
 			(effects
@@
 			)
 		)
-		(property "Footprint" "Diode_SMD:D_0402_1005Metric_Pad0.77x0.64mm_HandSolder"
+		(property "Footprint" "ScottoKeebs_Components:Diode_SOD-123"
 			(at 91.44 88.9 0)
 			(effects
@@
 			)
 		)
-		(property "Footprint" "Diode_SMD:D_0402_1005Metric_Pad0.77x0.64mm_HandSolder"
+		(property "Footprint" "ScottoKeebs_Components:Diode_SOD-123"
 			(at 91.44 120.65 0)
 			(effects
@@
 			)
 		)
-		(property "Footprint" "Diode_SMD:D_0402_1005Metric_Pad0.77x0.64mm_HandSolder"
+		(property "Footprint" "ScottoKeebs_Components:Diode_SOD-123"
 			(at 91.44 40.64 0)
 			(effects
@@
 			)
 		)
-		(property "Footprint" "Diode_SMD:D_0402_1005Metric_Pad0.77x0.64mm_HandSolder"
+		(property "Footprint" "ScottoKeebs_Components:Diode_SOD-123"
 			(at 73.66 55.88 0)
 			(effects
@@
 			)
 		)
-		(property "Footprint" "Diode_SMD:D_0402_1005Metric_Pad0.77x0.64mm_HandSolder"
+		(property "Footprint" "ScottoKeebs_Components:Diode_SOD-123"
 			(at 55.88 88.9 0)
 			(effects
@@
 			)
 		)
-		(property "Footprint" "Diode_SMD:D_0402_1005Metric_Pad0.77x0.64mm_HandSolder"
+		(property "Footprint" "ScottoKeebs_Components:Diode_SOD-123"
 			(at 55.88 72.39 0)
 			(effects
@@
 			)
 		)
-		(property "Footprint" "Diode_SMD:D_0402_1005Metric_Pad0.77x0.64mm_HandSolder"
+		(property "Footprint" "ScottoKeebs_Components:Diode_SOD-123"
 			(at 73.66 88.9 0)
 			(effects
@@
 			)
 		)
-		(property "Footprint" "Diode_SMD:D_0402_1005Metric_Pad0.77x0.64mm_HandSolder"
+		(property "Footprint" "ScottoKeebs_Components:Diode_SOD-123"
 			(at 91.44 105.41 0)
 			(effects
@@
 			)
 		)
-		(property "Footprint" "Diode_SMD:D_0402_1005Metric_Pad0.77x0.64mm_HandSolder"
+		(property "Footprint" "ScottoKeebs_Components:Diode_SOD-123"
 			(at 55.88 40.64 0)
 			(effects
@@
 			)
 		)
-		(property "Footprint" "Diode_SMD:D_0402_1005Metric_Pad0.77x0.64mm_HandSolder"
+		(property "Footprint" "ScottoKeebs_Components:Diode_SOD-123"
 			(at 55.88 105.41 0)
 			(effects
@@
 			)
 		)
-		(property "Footprint" "Diode_SMD:D_0402_1005Metric_Pad0.77x0.64mm_HandSolder"
+		(property "Footprint" "ScottoKeebs_Components:Diode_SOD-123"
 			(at 91.44 55.88 0)
 			(effects
@@
 			)
 		)
-		(property "Footprint" "Diode_SMD:D_0402_1005Metric_Pad0.77x0.64mm_HandSolder"
+		(property "Footprint" "ScottoKeebs_Components:Diode_SOD-123"
 			(at 109.22 40.64 0)
 			(effects
@@
 			)
 		)
-		(property "Footprint" "Diode_SMD:D_0402_1005Metric_Pad0.77x0.64mm_HandSolder"
+		(property "Footprint" "ScottoKeebs_Components:Diode_SOD-123"
 			(at 73.66 105.41 0)
 			(effects

Commit message: Pulled A10 to ground; found that a BlackPill dev board wo'nt DFU properly without it. Updated SK6812MINI-E footprint to be a rotated one; track layout stays the same, but the old footprint was incorrect, resulting in all key LEDs shorting out
Parts:
- LED1, LED10, LED11, LED12, LED13, LED14, LED15, LED16, LED17, LED18, LED19, LED2, LED20, LED21, LED3, LED4, LED5, LED6, LED7, LED8, LED9: footprint kicad-keyboard-parts:MX_SK6812MINI-E_REV -> kicad-keyboard-parts:MX_SK6812MINI-E_REV_ROTATED; symbol LED:SK6812MINI-E -> kicad-keyboard-parts:SK6812MINI-E
Connections:
- net GND: now also LED1.3 (VSS), LED10.3 (VSS), LED11.3 (VSS), LED12.3 (VSS), LED13.3 (VSS), LED14.3 (VSS), LED15.3 (VSS), LED16.3 (VSS), LED17.3 (VSS), LED18.3 (VSS), LED19.3 (VSS), LED2.3 (VSS), LED20.3 (VSS), LED21.3 (VSS), LED3.3 (VSS), LED4.3 (VSS), LED5.3 (VSS), LED6.3 (VSS), LED7.3 (VSS), LED8.3 (VSS), LED9.3 (VSS); no longer LED1.1 (VSS), LED10.1 (VSS), LED11.1 (VSS), LED12.1 (VSS), LED13.1 (VSS), LED14.1 (VSS), LED15.1 (VSS), LED16.1 (VSS), LED17.1 (VSS), LED18.1 (VSS), LED19.1 (VSS), LED2.1 (VSS), LED20.1 (VSS), LED21.1 (VSS), LED3.1 (VSS), LED4.1 (VSS), LED5.1 (VSS), LED6.1 (VSS), LED7.1 (VSS), LED8.1 (VSS), LED9.1 (VSS)
- net LED_DATA: now also LED1.4 (DIN); no longer LED1.2 (DIN)
- net LED_TO_UNDER: now also LED21.2 (DOUT); no longer LED21.4 (DOUT)
- net VBUS: now also LED1.1 (VDD), LED10.1 (VDD), LED11.1 (VDD), LED12.1 (VDD), LED13.1 (VDD), LED14.1 (VDD), LED15.1 (VDD), LED16.1 (VDD), LED17.1 (VDD), LED18.1 (VDD), LED19.1 (VDD), LED2.1 (VDD), LED20.1 (VDD), LED21.1 (VDD), LED3.1 (VDD), LED4.1 (VDD), LED5.1 (VDD), LED6.1 (VDD), LED7.1 (VDD), LED8.1 (VDD), LED9.1 (VDD); no longer LED1.3 (VDD), LED10.3 (VDD), LED11.3 (VDD), LED12.3 (VDD), LED13.3 (VDD), LED14.3 (VDD), LED15.3 (VDD), LED16.3 (VDD), LED17.3 (VDD), LED18.3 (VDD), LED19.3 (VDD), LED2.3 (VDD), LED20.3 (VDD), LED21.3 (VDD), LED3.3 (VDD), LED4.3 (VDD), LED5.3 (VDD), LED6.3 (VDD), LED7.3 (VDD), LED8.3 (VDD), LED9.3 (VDD)
- net at LED11.2 (DOUT): now also LED12.4 (DIN); no longer LED10.4 (DOUT)
- net at LED11.4 (DIN): now also LED10.2 (DOUT); no longer LED12.2 (DIN)
- net at LED8.2 (DOUT): now also LED9.4 (DIN); no longer LED7.4 (DOUT)
- net at LED8.4 (DIN): now also LED7.2 (DOUT); no longer LED9.2 (DIN)
- net at LED13.2 (DOUT): now also LED14.4 (DIN); no longer LED12.4 (DOUT)
- net at LED13.4 (DIN): now also LED12.2 (DOUT); no longer LED14.2 (DIN)
- net at LED16.2 (DOUT): now also LED17.4 (DIN); no longer LED15.4 (DOUT)
- net at LED16.4 (DIN): now also LED15.2 (DOUT); no longer LED17.2 (DIN)
- net at LED3.2 (DOUT): now also LED4.4 (DIN); no longer LED2.4 (DOUT)
- net at LED3.4 (DIN): now also LED2.2 (DOUT); no longer LED4.2 (DIN)
- net at LED20.2 (DOUT): now also LED21.4 (DIN); no longer LED19.4 (DOUT)
- net at LED20.4 (DIN): now also LED19.2 (DOUT); no longer LED21.2 (DIN)
- net at LED5.2 (DOUT): now also LED6.4 (DIN); no longer LED4.4 (DOUT)
- net at LED5.4 (DIN): now also LED4.2 (DOUT); no longer LED6.2 (DIN)
- net at LED18.2 (DOUT): now also LED19.4 (DIN); no longer LED17.4 (DOUT)
- net at LED18.4 (DIN): now also LED17.2 (DOUT); no longer LED19.2 (DIN)
- new net: LED10.4 (DIN), LED9.2 (DOUT)
- new net: LED14.2 (DOUT), LED15.4 (DIN)
- new net: LED6.2 (DOUT), LED7.4 (DIN)
- new net: LED1.2 (DOUT), LED2.4 (DIN)
Changed lines of the file:
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@@
 	)
 	(symbol
-		(lib_id "LED:SK6812MINI-E")
+		(lib_id "kicad-keyboard-parts:SK6812MINI-E")
 		(at 189.23 77.47 180)
 		(unit 1)
@@
 			)
 		)
-		(property "Footprint" "kicad-keyboard-parts:MX_SK6812MINI-E_REV"
+		(property "Footprint" "kicad-keyboard-parts:MX_SK6812MINI-E_REV_ROTATED"
 			(at 187.96 69.85 0)
 			(effects
@@
 	)
 	(symbol
-		(lib_id "LED:SK6812MINI-E")
+		(lib_id "kicad-keyboard-parts:SK6812MINI-E")
 		(at 148.59 97.79 0)
 		(unit 1)
@@
 			)
 		)
-		(property "Footprint" "kicad-keyboard-parts:MX_SK6812MINI-E_REV"
+		(property "Footprint" "kicad-keyboard-parts:MX_SK6812MINI-E_REV_ROTATED"
 			(at 149.86 105.41 0)
 			(effects
@@
 	)
 	(symbol
-		(lib_id "LED:SK6812MINI-E")
+		(lib_id "kicad-keyboard-parts:SK6812MINI-E")
 		(at 148.59 77.47 180)
 		(unit 1)
@@
 			)
 		)
-		(property "Footprint" "kicad-keyboard-parts:MX_SK6812MINI-E_REV"
+		(property "Footprint" "kicad-keyboard-parts:MX_SK6812MINI-E_REV_ROTATED"
 			(at 147.32 69.85 0)
 			(effects
@@
 	)
 	(symbol
-		(lib_id "LED:SK6812MINI-E")
+		(lib_id "kicad-keyboard-parts:SK6812MINI-E")
 		(at 189.23 55.88 0)
 		(unit 1)
@@
 			)
 		)
-		(property "Footprint" "kicad-keyboard-parts:MX_SK6812MINI-E_REV"
+		(property "Footprint" "kicad-keyboard-parts:MX_SK6812MINI-E_REV_ROTATED"
 			(at 190.5 63.5 0)
 			(effects
@@
 	)
 	(symbol
-		(lib_id "LED:SK6812MINI-E")
+		(lib_id "kicad-keyboard-parts:SK6812MINI-E")
 		(at 189.23 143.51 180)
 		(unit 1)
@@
 			)
 		)
-		(property "Footprint" "kicad-keyboard-parts:MX_SK6812MINI-E_REV"
+		(property "Footprint" "kicad-keyboard-parts:MX_SK6812MINI-E_REV_ROTATED"
 			(at 187.96 135.89 0)
 			(effects
@@
 	)
 	(symbol
-		(lib_id "LED:SK6812MINI-E")
+		(lib_id "kicad-keyboard-parts:SK6812MINI-E")
 		(at 168.91 29.21 180)
 		(unit 1)
@@
 			)
 		)
-		(property "Footprint" "kicad-keyboard-parts:MX_SK6812MINI-E_REV"
+		(property "Footprint" "kicad-keyboard-parts:MX_SK6812MINI-E_REV_ROTATED"
 			(at 167.64 21.59 0)
 			(effects
@@
 	)
 	(symbol
-		(lib_id "LED:SK6812MINI-E")
+		(lib_id "kicad-keyboard-parts:SK6812MINI-E")
 		(at 168.91 97.79 0)
 		(unit 1)
@@
 			)
 		)
-		(property "Footprint" "kicad-keyboard-parts:MX_SK6812MINI-E_REV"
+		(property "Footprint" "kicad-keyboard-parts:MX_SK6812MINI-E_REV_ROTATED"
 			(at 170.18 105.41 0)
 			(effects
@@
 	)
 	(symbol
-		(lib_id "LED:SK6812MINI-E")
+		(lib_id "kicad-keyboard-parts:SK6812MINI-E")
 		(at 189.23 97.79 0)
 		(unit 1)
@@
 			)
 		)
-		(property "Footprint" "kicad-keyboard-parts:MX_SK6812MINI-E_REV"
+		(property "Footprint" "kicad-keyboard-parts:MX_SK6812MINI-E_REV_ROTATED"
 			(at 190.5 105.41 0)
 			(effects
@@
 	)
 	(symbol
-		(lib_id "LED:SK6812MINI-E")
+		(lib_id "kicad-keyboard-parts:SK6812MINI-E")
 		(at 189.23 119.38 180)
 		(unit 1)
@@
 			)
 		)
-		(property "Footprint" "kicad-keyboard-parts:MX_SK6812MINI-E_REV"
+		(property "Footprint" "kicad-keyboard-parts:MX_SK6812MINI-E_REV_ROTATED"
 			(at 187.96 111.76 0)
 			(effects
@@
 	)
 	(symbol
-		(lib_id "LED:SK6812MINI-E")
+		(lib_id "kicad-keyboard-parts:SK6812MINI-E")
 		(at 168.91 55.88 0)
 		(unit 1)
@@
 			)
 		)
-		(property "Footprint" "kicad-keyboard-parts:MX_SK6812MINI-E_REV"
+		(property "Footprint" "kicad-keyboard-parts:MX_SK6812MINI-E_REV_ROTATED"
 			(at 170.18 63.5 0)
 			(effects
@@
 	)
 	(symbol
-		(lib_id "LED:SK6812MINI-E")
+		(lib_id "kicad-keyboard-parts:SK6812MINI-E")
 		(at 148.59 119.38 180)
 		(unit 1)
@@
 			)
 		)
-		(property "Footprint" "kicad-keyboard-parts:MX_SK6812MINI-E_REV"
+		(property "Footprint" "kicad-keyboard-parts:MX_SK6812MINI-E_REV_ROTATED"
 			(at 147.32 111.76 0)
 			(effects
@@
 	)
 	(symbol
-		(lib_id "LED:SK6812MINI-E")
+		(lib_id "kicad-keyboard-parts:SK6812MINI-E")
 		(at 158.75 143.51 180)
 		(unit 1)
@@
 			)
 		)
-		(property "Footprint" "kicad-keyboard-parts:MX_SK6812MINI-E_REV"
+		(property "Footprint" "kicad-keyboard-parts:MX_SK6812MINI-E_REV_ROTATED"
 			(at 157.48 135.89 0)
 			(effects
@@
 	)
 	(symbol
-		(lib_id "LED:SK6812MINI-E")
+		(lib_id "kicad-keyboard-parts:SK6812MINI-E")
 		(at 213.36 87.63 270)
 		(unit 1)
@@
 			)
 		)
-		(property "Footprint" "kicad-keyboard-parts:MX_SK6812MINI-E_REV"
+		(property "Footprint" "kicad-keyboard-parts:MX_SK6812MINI-E_REV_ROTATED"
 			(at 205.74 88.9 0)
 			(effects
@@
 	)
 	(symbol
-		(lib_id "LED:SK6812MINI-E")
+		(lib_id "kicad-keyboard-parts:SK6812MINI-E")
 		(at 213.36 55.88 0)
 		(unit 1)
@@
 			)
 		)
-		(property "Footprint" "kicad-keyboard-parts:MX_SK6812MINI-E_REV"
+		(property "Footprint" "kicad-keyboard-parts:MX_SK6812MINI-E_REV_ROTATED"
 			(at 214.63 63.5 0)
 			(effects
@@
 	)
 	(symbol
-		(lib_id "LED:SK6812MINI-E")
+		(lib_id "kicad-keyboard-parts:SK6812MINI-E")
 		(at 189.23 29.21 180)
 		(unit 1)
@@
 			)
 		)
-		(property "Footprint" "kicad-keyboard-parts:MX_SK6812MINI-E_REV"
+		(property "Footprint" "kicad-keyboard-parts:MX_SK6812MINI-E_REV_ROTATED"
 			(at 187.96 21.59 0)
 			(effects
@@
 	)
 	(symbol
-		(lib_id "LED:SK6812MINI-E")
+		(lib_id "kicad-keyboard-parts:SK6812MINI-E")
 		(at 148.59 29.21 180)
 		(unit 1)
@@
 			)
 		)
-		(property "Footprint" "kicad-keyboard-parts:MX_SK6812MINI-E_REV"
+		(property "Footprint" "kicad-keyboard-parts:MX_SK6812MINI-E_REV_ROTATED"
 			(at 147.32 21.59 0)
 			(effects
@@
 	)
 	(symbol
-		(lib_id "LED:SK6812MINI-E")
+		(lib_id "kicad-keyboard-parts:SK6812MINI-E")
 		(at 168.91 119.38 180)
 		(unit 1)
@@
 			)
 		)
-		(property "Footprint" "kicad-keyboard-parts:MX_SK6812MINI-E_REV"
+		(property "Footprint" "kicad-keyboard-parts:MX_SK6812MINI-E_REV_ROTATED"
 			(at 167.64 111.76 0)
 			(effects
@@
 	)
 	(symbol
-		(lib_id "LED:SK6812MINI-E")
+		(lib_id "kicad-keyboard-parts:SK6812MINI-E")
 		(at 213.36 128.27 270)
 		(unit 1)
@@
 			)
 		)
-		(property "Footprint" "kicad-keyboard-parts:MX_SK6812MINI-E_REV"
+		(property "Footprint" "kicad-keyboard-parts:MX_SK6812MINI-E_REV_ROTATED"
 			(at 205.74 129.54 0)
 			(effects
@@
 	)
 	(symbol
-		(lib_id "LED:SK6812MINI-E")
+		(lib_id "kicad-keyboard-parts:SK6812MINI-E")
 		(at 213.36 29.21 180)
 		(unit 1)
@@
 			)
 		)
-		(property "Footprint" "kicad-keyboard-parts:MX_SK6812MINI-E_REV"
+		(property "Footprint" "kicad-keyboard-parts:MX_SK6812MINI-E_REV_ROTATED"
 			(at 212.09 21.59 0)
 			(effects
@@
 	)
 	(symbol
-		(lib_id "LED:SK6812MINI-E")
+		(lib_id "kicad-keyboard-parts:SK6812MINI-E")
 		(at 168.91 77.47 180)
 		(unit 1)
@@
 			)
 		)
-		(property "Footprint" "kicad-keyboard-parts:MX_SK6812MINI-E_REV"
+		(property "Footprint" "kicad-keyboard-parts:MX_SK6812MINI-E_REV_ROTATED"
 			(at 167.64 69.85 0)
 			(effects
@@
 	)
 	(symbol
-		(lib_id "LED:SK6812MINI-E")
+		(lib_id "kicad-keyboard-parts:SK6812MINI-E")
 		(at 148.59 55.88 0)
 		(unit 1)
@@
 			)
 		)
-		(property "Footprint" "kicad-keyboard-parts:MX_SK6812MINI-E_REV"
+		(property "Footprint" "kicad-keyboard-parts:MX_SK6812MINI-E_REV_ROTATED"
 			(at 149.86 63.5 0)
 			(effects
